File: PCB/PedalFX2/PedalFX2.sch (KiCad schematic (older format))
At the start: 11 parts, among them J1 Conn_01x04_Female, T1 ACJS-MHDR, T2 ACJS-MHDR, T3 54-00129

Commit message: Goofed
Goofed internal connector flipped and jacks not flush with housing. All fixed now, all boards redone.
Parts:
- added SP3: Hammond_1590B, AVR-KiCAD-Lib-Special:1590B, symbol Special:Hammond_1590B
Connections:
- net BYPASS: now reaches SP1.1, SP1.2
- net Pedal_OUT: now reaches SP1.5, T2.6 (T)
- net OUT: now reaches J1.4 (Pin_4), R3.1, SP1.8
- net Pedal_IN: now reaches SP1.4, T1.6 (T)
- net IN: now reaches J1.1 (Pin_1), R2.1, SP1.3, SP1.7
Other:
- moved on the sheet: T1, T2
Changed lines of the file:
@@
 L Connectors:ACJS-MHDR T1
 U 1 1 5D0841AB
-P 3900 2900
-F 0 "T1" H 3583 3265 50  0000 C CNN
-F 1 "ACJS-MHDR" H 3583 3174 50  0000 C CNN
-F 2 "AVR-KiCAD-Lib-Connectors:ACJS-MHDR" H 3800 4400 50  0001 C CNN
-F 3 "" H 3900 4500 50  0001 C CNN
-F 4 "1.41000" H 4100 4650 50  0001 C CNN "Cost QTY: 1"
-F 5 "0.81420" H 4200 4750 50  0001 C CNN "Cost QTY: 1000"
-F 6 "0.74520" H 4300 4850 50  0001 C CNN "Cost QTY: 2500"
-F 7 "*" H 4400 4950 50  0001 C CNN "Cost QTY: 5000"
-F 8 "*" H 4500 5050 50  0001 C CNN "Cost QTY: 10000"
-F 9 "Amphenol Sine Systems Corp" H 4600 5150 50  0001 C CNN "MFR"
-F 10 "ACJS-MHDR" H 4700 5250 50  0001 C CNN "MFR#"
-F 11 "Digikey" H 4800 5350 50  0001 C CNN "Vendor"
-F 12 "889-1817-ND" H 4900 5450 50  0001 C CNN "Vendor #"
-F 13 "AVR" H 5000 5550 50  0001 C CNN "Designer"
-F 14 "12.7mm" H 5100 5650 50  0001 C CNN "Height"
-F 15 "1/5/2019" H 6200 6750 50  0001 C CNN "Date Created"
-F 16 "1/5/2019" H 5200 5750 50  0001 C CNN "Date Modified"
-F 17 "Yes" H 5300 5850 50  0001 C CNN "Lead-Free ?"
-F 18 "RoHS 1" H 5400 5950 50  0001 C CNN "RoHS Levels"
-F 19 "ThroughHole" H 5500 6050 50  0001 C CNN "Mounting"
-F 20 "6" H 5600 6150 50  0001 C CNN "Pin Count #"
-F 21 "Active" H 5700 6250 50  0001 C CNN "Status"
-F 22 "*" H 5800 6350 50  0001 C CNN "Tolerance"
-F 23 "TRS Connector 6.35mm" H 5900 6450 50  0001 C CNN "Type"
-F 24 "*" H 6000 6550 50  0001 C CNN "Voltage"
-F 25 "*" H 6100 6700 50  0001 C CNN "Package"
-F 26 "CONN JACK STEREO 1/4\" R/A" H 6500 7100 50  0001 C CNN "Description"
-F 27 "ACJS-MHDR" H 6300 6900 50  0001 C CNN "_Value_"
-F 28 "*" H 6400 7000 50  0001 C CNN "Management_ID"
-	1    3900 2900
+P 3450 2900
+F 0 "T1" H 2600 3150 50  0000 C CNN
+F 1 "ACJS-MHDR" H 3250 3150 50  0000 C CNN
+F 2 "AVR-KiCAD-Lib-Connectors:ACJS-MHDR" H 3350 4400 50  0001 C CNN
+F 3 "" H 3450 4500 50  0001 C CNN
+F 4 "1.41000" H 3650 4650 50  0001 C CNN "Cost QTY: 1"
+F 5 "0.81420" H 3750 4750 50  0001 C CNN "Cost QTY: 1000"
+F 6 "0.74520" H 3850 4850 50  0001 C CNN "Cost QTY: 2500"
+F 7 "*" H 3950 4950 50  0001 C CNN "Cost QTY: 5000"
+F 8 "*" H 4050 5050 50  0001 C CNN "Cost QTY: 10000"
+F 9 "Amphenol Sine Systems Corp" H 4150 5150 50  0001 C CNN "MFR"
+F 10 "ACJS-MHDR" H 4250 5250 50  0001 C CNN "MFR#"
+F 11 "Digikey" H 4350 5350 50  0001 C CNN "Vendor"
+F 12 "889-1817-ND" H 4450 5450 50  0001 C CNN "Vendor #"
+F 13 "AVR" H 4550 5550 50  0001 C CNN "Designer"
+F 14 "12.7mm" H 4650 5650 50  0001 C CNN "Height"
+F 15 "1/5/2019" H 5750 6750 50  0001 C CNN "Date Created"
+F 16 "1/5/2019" H 4750 5750 50  0001 C CNN "Date Modified"
+F 17 "Yes" H 4850 5850 50  0001 C CNN "Lead-Free ?"
+F 18 "RoHS 1" H 4950 5950 50  0001 C CNN "RoHS Levels"
+F 19 "ThroughHole" H 5050 6050 50  0001 C CNN "Mounting"
+F 20 "6" H 5150 6150 50  0001 C CNN "Pin Count #"
+F 21 "Active" H 5250 6250 50  0001 C CNN "Status"
+F 22 "*" H 5350 6350 50  0001 C CNN "Tolerance"
+F 23 "TRS Connector 6.35mm" H 5450 6450 50  0001 C CNN "Type"
+F 24 "*" H 5550 6550 50  0001 C CNN "Voltage"
+F 25 "*" H 5650 6700 50  0001 C CNN "Package"
+F 26 "CONN JACK STEREO 1/4\" R/A" H 6050 7100 50  0001 C CNN "Description"
+F 27 "ACJS-MHDR" H 5850 6900 50  0001 C CNN "_Value_"
+F 28 "*" H 5950 7000 50  0001 C CNN "Management_ID"
+	1    3450 2900
 	1    0    0    -1
 $EndComp
@@
 L Connectors:ACJS-MHDR T2
 U 1 1 5D086FC4
-P 7600 2900
-F 0 "T2" H 7600 3150 50  0000 R CNN
-F 1 "ACJS-MHDR" H 7600 2300 50  0000 R CNN
-F 2 "AVR-KiCAD-Lib-Connectors:ACJS-MHDR" H 7500 4400 50  0001 C CNN
-F 3 "" H 7600 4500 50  0001 C CNN
-F 4 "1.41000" H 7800 4650 50  0001 C CNN "Cost QTY: 1"
-F 5 "0.81420" H 7900 4750 50  0001 C CNN "Cost QTY: 1000"
-F 6 "0.74520" H 8000 4850 50  0001 C CNN "Cost QTY: 2500"
-F 7 "*" H 8100 4950 50  0001 C CNN "Cost QTY: 5000"
-F 8 "*" H 8200 5050 50  0001 C CNN "Cost QTY: 10000"
-F 9 "Amphenol Sine Systems Corp" H 8300 5150 50  0001 C CNN "MFR"
-F 10 "ACJS-MHDR" H 8400 5250 50  0001 C CNN "MFR#"
-F 11 "Digikey" H 8500 5350 50  0001 C CNN "Vendor"
-F 12 "889-1817-ND" H 8600 5450 50  0001 C CNN "Vendor #"
-F 13 "AVR" H 8700 5550 50  0001 C CNN "Designer"
-F 14 "12.7mm" H 8800 5650 50  0001 C CNN "Height"
-F 15 "1/5/2019" H 9900 6750 50  0001 C CNN "Date Created"
-F 16 "1/5/2019" H 8900 5750 50  0001 C CNN "Date Modified"
-F 17 "Yes" H 9000 5850 50  0001 C CNN "Lead-Free ?"
-F 18 "RoHS 1" H 9100 5950 50  0001 C CNN "RoHS Levels"
-F 19 "ThroughHole" H 9200 6050 50  0001 C CNN "Mounting"
-F 20 "6" H 9300 6150 50  0001 C CNN "Pin Count #"
-F 21 "Active" H 9400 6250 50  0001 C CNN "Status"
-F 22 "*" H 9500 6350 50  0001 C CNN "Tolerance"
-F 23 "TRS Connector 6.35mm" H 9600 6450 50  0001 C CNN "Type"
-F 24 "*" H 9700 6550 50  0001 C CNN "Voltage"
-F 25 "*" H 9800 6700 50  0001 C CNN "Package"
-F 26 "CONN JACK STEREO 1/4\" R/A" H 10200 7100 50  0001 C CNN "Description"
-F 27 "ACJS-MHDR" H 10000 6900 50  0001 C CNN "_Value_"
-F 28 "*" H 10100 7000 50  0001 C CNN "Management_ID"
-	1    7600 2900
+P 7900 2900
+F 0 "T2" H 7900 3150 50  0000 R CNN
+F 1 "ACJS-MHDR" H 7900 2300 50  0000 R CNN
+F 2 "AVR-KiCAD-Lib-Connectors:ACJS-MHDR" H 7800 4400 50  0001 C CNN
+F 3 "" H 7900 4500 50  0001 C CNN
+F 4 "1.41000" H 8100 4650 50  0001 C CNN "Cost QTY: 1"
+F 5 "0.81420" H 8200 4750 50  0001 C CNN "Cost QTY: 1000"
+F 6 "0.74520" H 8300 4850 50  0001 C CNN "Cost QTY: 2500"
+F 7 "*" H 8400 4950 50  0001 C CNN "Cost QTY: 5000"
+F 8 "*" H 8500 5050 50  0001 C CNN "Cost QTY: 10000"
+F 9 "Amphenol Sine Systems Corp" H 8600 5150 50  0001 C CNN "MFR"
+F 10 "ACJS-MHDR" H 8700 5250 50  0001 C CNN "MFR#"
+F 11 "Digikey" H 8800 5350 50  0001 C CNN "Vendor"
+F 12 "889-1817-ND" H 8900 5450 50  0001 C CNN "Vendor #"
+F 13 "AVR" H 9000 5550 50  0001 C CNN "Designer"
+F 14 "12.7mm" H 9100 5650 50  0001 C CNN "Height"
+F 15 "1/5/2019" H 10200 6750 50  0001 C CNN "Date Created"
+F 16 "1/5/2019" H 9200 5750 50  0001 C CNN "Date Modified"
+F 17 "Yes" H 9300 5850 50  0001 C CNN "Lead-Free ?"
+F 18 "RoHS 1" H 9400 5950 50  0001 C CNN "RoHS Levels"
+F 19 "ThroughHole" H 9500 6050 50  0001 C CNN "Mounting"
+F 20 "6" H 9600 6150 50  0001 C CNN "Pin Count #"
+F 21 "Active" H 9700 6250 50  0001 C CNN "Status"
+F 22 "*" H 9800 6350 50  0001 C CNN "Tolerance"
+F 23 "TRS Connector 6.35mm" H 9900 6450 50  0001 C CNN "Type"
+F 24 "*" H 10000 6550 50  0001 C CNN "Voltage"
+F 25 "*" H 10100 6700 50  0001 C CNN "Package"
+F 26 "CONN JACK STEREO 1/4\" R/A" H 10500 7100 50  0001 C CNN "Description"
+F 27 "ACJS-MHDR" H 10300 6900 50  0001 C CNN "_Value_"
+F 28 "*" H 10400 7000 50  0001 C CNN "Management_ID"
+	1    7900 2900
 	-1   0    0    -1
 $EndComp
@@
 $EndComp
 Wire Wire Line
-	4350 3300 4100 3300
+	4350 3300 3650 3300
 $Comp
 L power:GND #PWR02
@@
 $EndComp
 Wire Wire Line
-	4100 2800 5100 2800
+	3650 2800 5100 2800
 Wire Wire Line
 	5100 2800 5100 2900
 Wire Wire Line
-	7400 3300 7100 3300
+	7700 3300 7100 3300
 $Comp
 L power:GND #PWR07
@@
 $EndComp
 Wire Wire Line
-	7400 2800 6300 2800
+	7700 2800 6300 2800
 Wire Wire Line
 	6300 2800 6300 2900
@@
 Wire Wire Line
 	4950 3400 5150 3400
-Text Notes 3150 3600 0    50   ~ 0
+Text Notes 2600 3550 0    50   ~ 0
 Guitar Input
-Text Notes 7450 3750 0    50   ~ 0
+Text Notes 7500 3600 0    50   ~ 0
 Output To Amp or Next Pedal
 Text Notes 5200 4550 0    50   ~ 0
@@
 Wire Wire Line
 	7450 4750 8350 4750
-Text Notes 7350 4600 0    50   ~ 0
+Text Notes 7900 5300 0    50   ~ 0
 DC Power In and Filtering
+$Comp
+L Special:Hammond_1590B SP3
+U 1 1 5CD9AC8E
+P 2600 3850
+F 0 "SP3" H 2600 3900 50  0000 L CNN
+F 1 "Hammond_1590B" H 2600 3300 50  0000 L CNN
+F 2 "AVR-KiCAD-Lib-Special:1590B" H 2650 4000 50  0001 C CNN
+F 3 "https://www.hammfg.com/electronics/small-case/diecast/1590.pdf" H 2600 3850 50  0001 C CNN
+F 4 "8.34000" H 2700 4100 50  0001 C CNN "Cost QTY: 1"
+F 5 "5.54610" H 2800 4200 50  0001 C CNN "Cost QTY: 1000"
+F 6 "*" H 2900 4300 50  0001 C CNN "Cost QTY: 2500"
+F 7 "*" H 3000 4400 50  0001 C CNN "Cost QTY: 5000"
+F 8 "*" H 3100 4500 50  0001 C CNN "Cost QTY: 10000"
+F 9 "Hammond Manufacturing" H 3200 4600 50  0001 C CNN "MFR"
+F 10 "1590B" H 3300 4700 50  0001 C CNN "MFR#"
+F 11 "Digikey" H 3400 4800 50  0001 C CNN "Vendor"
+F 12 "HM151-ND" H 3500 4900 50  0001 C CNN "Vendor #"
+F 13 "AVR" H 3600 5000 50  0001 C CNN "Designer"
+F 14 "30.99mm" H 3700 5100 50  0001 C CNN "Height"
+F 15 "5/9/2019" H 4800 6200 50  0001 C CNN "Date Created"
+F 16 "5/9/2019" H 3800 5200 50  0001 C CNN "Date Modified"
+F 17 "Yes" H 3900 5300 50  0001 C CNN "Lead-Free ?"
+F 18 "1" H 4000 5400 50  0001 C CNN "RoHS Levels"
+F 19 "*" H 4100 5500 50  0001 C CNN "Mounting"
+F 20 "*" H 4200 5600 50  0001 C CNN "Pin Count #"
+F 21 "*" H 4300 5700 50  0001 C CNN "Status"
+F 22 "*" H 4400 5800 50  0001 C CNN "Tolerance"
+F 23 "Enclosure, Cast Aluminum" H 4500 5900 50  0001 C CNN "Type"
+F 24 "*" H 4600 6000 50  0001 C CNN "Voltage"
+F 25 "*" H 4700 6150 50  0001 C CNN "Package"
+F 26 "BOX ALUM UNPAINTED 4.41\"LX2.38\"W" H 5000 6450 50  0001 C CNN "Description"
+F 27 "1590B" H 4900 6350 50  0001 C CNN "_Value_"
+F 28 "*" H 5000 6450 50  0001 C CNN "Management_ID"
+	1    2600 3850
+	1    0    0    -1
+$EndComp
+Text Label 5350 3400 0    50   ~ 0
+IN
+Text Label 6000 3400 0    50   ~ 0
+OUT
+Text Label 7150 3300 0    50   ~ 0
+Pedal_OUT
+Text Label 3750 3300 0    50   ~ 0
+Pedal_IN
+Text Label 5550 3250 0    50   ~ 0
+BYPASS
 $EndSCHEMATC
