File: PCB/PedalFX2 - 1590BB/PedalFX2_1590BB.kicad_pcb (KiCad board)
At the start: 2 copper layers, 109.5 x 40.1 mm, 12 parts, among them J1 Conn_01x04_Female, T1 ACJS-MHDR, T2 ACJS-MHDR, T3 54-00129

Commit message: Goofed
Goofed internal connector flipped and jacks not flush with housing. All fixed now, all boards redone.
Parts:
- moved C2 8.45 mm to (183.6, 137.2)
- moved J1 7.60 mm to (158.6, 111.7), turned to 270 degrees
- moved T1 4.40 mm to (201.5, 122.6)
- moved T2 4.40 mm to (108.0, 122.6)
- moved SP2 3.72 mm to (139.8, 139.5)
- moved C1 2.35 mm to (188.9, 138.2)
Connections:
- net Net-(J1-Pad1) renamed /IN
- net Net-(J1-Pad4) renamed /OUT
- net Net-(SP1-Pad1) renamed /BYPASS
- net Net-(SP1-Pad4) renamed /Pedal_IN
- net Net-(SP1-Pad5) renamed /Pedal_OUT
Routing:
- net /OUT: track 113.7 -> 51.4 mm
- net /IN: track 105.0 -> 55.7 mm
- net +9V: track 124.2 -> 115.4 mm, vias 2 -> 1
- net /Pedal_IN: track 46.3 -> 50.7 mm
- net /Pedal_OUT: track 44.0 -> 47.6 mm
- net Net-(R1-Pad2): track 5.15 -> 4.20 mm
- added copper zone on F.Cu, net GND
Other:
- board size 109.5 x 40.1 mm -> 114.5 x 40.1 mm

Commit message: Templates
Added pedal templates for each size of PedalFX2
Changed lines of the file:
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@@
     )
   )
+  (gr_line (start 149.15 109.9) (end 154.75 109.9) (layer Edge.Cuts) (width 0.2))
+  (gr_line (start 160.35 109.9) (end 154.75 109.9) (layer Edge.Cuts) (width 0.2))
   (gr_line (start 202.3 142.8) (end 202.3 149.8) (layer Margin) (width 0.15))
   (gr_line (start 211.8 142.8) (end 202.3 142.8) (layer Margin) (width 0.15))
@@
   (gr_line (start 146.65 113) (end 97.5 113) (layer Edge.Cuts) (width 0.2))
   (gr_line (start 162.85 113) (end 212 113) (layer Edge.Cuts) (width 0.2))
-  (gr_line (start 154.75 109.9) (end 149.15 109.9) (layer Edge.Cuts) (width 0.2))
-  (gr_line (start 154.75 109.9) (end 160.35 109.9) (layer Edge.Cuts) (width 0.2))
   (gr_line (start 146.65 113) (end 149.15 109.9) (layer Edge.Cuts) (width 0.2))
   (gr_line (start 160.35 109.9) (end 162.85 113) (layer Edge.Cuts) (width 0.2))
