File: PCB/PedalFX2 - 1590N1/PedalFX2_1590N1.kicad_pcb (KiCad board)
At the start: 2 copper layers, 59 x 43.7 mm, 11 parts, among them J1 Conn_01x04_Female, T1 ACJS-MHDR, T2 ACJS-MHDR, T3 54-00129

Commit message: Various versions added and editted
Added 1590N1 size and 1590A has been editted.
Other:
- board text added: "9V"
- board text added: "FX_IN"
- board text added: "FX_OUT"
- board text added: "GND"
Changed lines of the file:
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@@
   (general
     (thickness 1.6)
-    (drawings 26)
+    (drawings 30)
     (tracks 71)
     (zones 0)
@@
     )
   )
+  (gr_text FX_OUT (at 121.8 124.45 90) (layer B.SilkS)
+    (effects (font (size 1 1) (thickness 0.15)) (justify mirror))
+  )
+  (gr_text 9V (at 124.25 122.85 90) (layer B.SilkS)
+    (effects (font (size 1 1) (thickness 0.15)) (justify mirror))
+  )
+  (gr_text GND (at 126.9 123.45 90) (layer B.SilkS)
+    (effects (font (size 1 1) (thickness 0.15)) (justify mirror))
+  )
+  (gr_text FX_IN (at 129.35 123.95 90) (layer B.SilkS)
+    (effects (font (size 1 1) (thickness 0.15)) (justify mirror))
+  )
   (gr_line (start 117.45 121.65) (end 96 121.65) (layer Edge.Cuts) (width 0.2))
